Commit message: Rename package to vector_the_arm_description (ROS-valid name)

File: finalAssem.SLDASM/urdf/vector_the_arm_description.urdf (robot description, URDF)
Before this commit: robot finalAssem.SLDASM, 5 links, 4 joints
Links:
- link Link1: geometry collision mesh filename=package://vector_the_arm_description/meshes/Link1.STL; visual mesh filename=package://vector_the_arm_description/meshes/Link1.STL
- link Link2: geometry collision mesh filename=package://vector_the_arm_description/meshes/Link2.STL; visual mesh filename=package://vector_the_arm_description/meshes/Link2.STL
- link Link3: geometry collision mesh filename=package://vector_the_arm_description/meshes/Link3.STL; visual mesh filename=package://vector_the_arm_description/meshes/Link3.STL
- link Link4: geometry collision mesh filename=package://vector_the_arm_description/meshes/Link4.STL; visual mesh filename=package://vector_the_arm_description/meshes/Link4.STL
- link base_link: geometry collision mesh filename=package://vector_the_arm_description/meshes/base_link.STL; visual mesh filename=package://vector_the_arm_description/meshes/base_link.STL
