Commit message: update joint state publisher and gui to run with simulated model and physical model at the same time WIP

File: ros2/src/vector_the_arm_description/urdf/vector_the_arm_description.urdf (robot description, URDF)
Before this commit: robot vector_the_arm_description, 5 links, 4 joints
Joints:
- joint Joint1: origin xyz=0 0 0 rpy=0 0 0 -> xyz=0 0 0 rpy=0 0 3.1416

Commit message: Added torque limit script and finished calibration for servo 5 and 6 - next step to integrate object detection

File: ros2/src/vector_the_arm_description/urdf/vector_the_arm_description.urdf (robot description, URDF)
Before this commit: robot vector_the_arm_description, 5 links, 4 joints
Links:
- added link Link5, mass 0.15471; collision mesh filename=package://vector_the_arm_description/meshes/Link5.STL; visual mesh filename=package://vector_the_arm_description/meshes/Link5.STL
- added link gripper, mass 0.020259; collision mesh filename=package://vector_the_arm_description/meshes/gripper.STL; visual mesh filename=package://vector_the_arm_description/meshes/gripper.STL
Joints:
- added joint Joint5: type continuous, parent Link4, child Link5, origin xyz=-0.1347 -0.000286 -0.022559 rpy=1.5708 0 1.5708, axis 0 0 1
- added joint gripper_joint: type revolute, parent Link5, child gripper, origin xyz=0.002823 0 -0.008531 rpy=1.5708 -1.5708 0, axis 0 0 1, limit lower=0 upper=2.126 effort=1.0 velocity=1.0

Commit message: update readme improve gripper support

File: ros2/src/vector_the_arm_description/urdf/vector_the_arm_description.urdf (robot description, URDF)
Before this commit: robot vector_the_arm_description, 7 links, 6 joints
Joints:
- joint gripper_joint: limit lower=0 upper=2.126 effort=1.0 velocity=1.0 -> lower=-0.468 upper=1.658 effort=1.0 velocity=1.0

File: ros2/src/vector_the_arm_moveit_config/config/vector_the_arm_description.ros2_control.xacro (robot description, xacro)
@@ -36,4 +36,18 @@
                 <state_interface name="velocity"/>
             </joint>
+            <joint name="Joint5">
+                <command_interface name="position"/>
+                <state_interface name="position">
+                  <param name="initial_value">${initial_positions['Joint5']}</param>
+                </state_interface>
+                <state_interface name="velocity"/>
+            </joint>
+            <joint name="gripper_joint">
+                <command_interface name="position"/>
+                <state_interface name="position">
+                  <param name="initial_value">${initial_positions['gripper_joint']}</param>
+                </state_interface>
+                <state_interface name="velocity"/>
+            </joint>
         </ros2_control>
     </xacro:macro>
